Commit message: [urdf] Create three situations urdf

File: urdf/chimera_bricks_detaching.urdf.xacro (robot description, xacro)
@@ -2,5 +2,4 @@
 <robot
     xmlns:xacro="http://www.ros.org/wiki/xacro" name="dragon" >
-  <!-- 1: pick_mode 2:docking_mode 3:detaching_mode -->
   <!--<xacro:arg name="fixed_grapple" default="true" />-->
   <!-- spot -->
@@ -16,4 +15,17 @@
     <child link="root" />
   </joint>
+  <joint name="end_effector_fixed_joint" type="fixed">
+    <parent link="link4"/>
+    <child link="end_effector_link"/>
+    <origin xyz="${link_length} 0 0" rpy="${0} ${pi/2} ${0}"/>
+  </joint>
+  <link name="end_effector_link">
+    <visual>
+      <origin xyz="0 0 0" rpy="0 0 0"/>
+      <geometry>
+	<mesh filename="package://chimera_ros/meshes/end_effector.dae" scale="1 1 1" />
+      </geometry>
+    </visual>
+  </link>
   <joint name="wall_fixed_joint" type="fixed">
     <parent link="base_link"/>
@@ -25,20 +37,7 @@
       <origin xyz="0 0 0" rpy="0 0 0"/>
       <geometry>
-	<mesh filename="package://chimera_ros/meshes/brick_wall_low.dae" scale="1 1 1" />
+	<mesh filename="package://chimera_ros/meshes/brick_wall_high.dae" scale="1 1 1" />
       </geometry>
     </visual>
   </link>
-  <joint name="end_effector_fixed_joint" type="fixed">
-    <parent link="link4"/>
-    <child link="end_effector_link"/>
-    <origin xyz="${link_length} 0 0" rpy="${0} ${pi/2} ${0}"/>
-  </joint>
-  <link name="end_effector_link">
-    <visual>
-     <origin xyz="0 0 0" rpy="0 0 0"/>
-     <geometry>
-       <mesh filename="package://chimera_ros/meshes/end_effector.dae" scale="1 1 1" />
-     </geometry>
-    </visual>
-  </link>
 </robot>

File: urdf/chimera_bricks_picking.urdf.xacro (robot description, xacro)
@@ -25,5 +25,5 @@
       <origin xyz="0 0 0" rpy="0 0 0"/>
       <geometry>
-	<mesh filename="package://chimera_ros/meshes/brick_wall_low.dae" scale="1 1 1" />
+	<mesh filename="package://chimera_ros/meshes/brick_picking.dae" scale="1 1 1" />
       </geometry>
     </visual>
