Commit message: [urdf] changed the used ground robot model

File: urdf/chimera_bricks_checking.urdf.xacro (robot description, xacro)
@@ -10,22 +10,23 @@
   <joint name="grapple_attachment_joint" type="fixed">
     <!-- <origin xyz="0.0 0.0 0.224" rpy="${pi} ${pi/2} 0" /> -->
-    <origin xyz="0.0 0.0 0.3" rpy="0 ${-pi/2} 0" />
+    <!-- <origin xyz="0.0 0.0 0.3" rpy="0 ${-pi/2} 0" />  -->
+    <origin xyz="0.0 0.0 0.0" rpy="0 ${-pi/2} 0" />
     <axis xyz="1 0 0" />
     <parent link="base_fixture" />
     <child link="root" />
   </joint>
-  <!-- <joint name="end_effector_fixed_joint" type="fixed"> -->
-  <!--   <parent link="link4"/> -->
-  <!--   <child link="end_effector_link"/> -->
-  <!--   <origin xyz="${link_length} 0 0" rpy="0 ${pi/2} 0"/> -->
-  <!-- </joint> -->
-  <!-- <link name="end_effector_link"> -->
-  <!--   <visual> -->
-  <!--     <origin xyz="0 0 0" rpy="0 0 0"/> -->
-  <!--     <geometry> -->
-  <!-- 	<mesh filename="package://chimera_ros/meshes/end_effector.dae" scale="1 1 1" /> -->
-  <!--     </geometry> -->
-  <!--   </visual> -->
-  <!-- </link> -->
+  <joint name="end_effector_fixed_joint" type="fixed">
+    <parent link="link4"/>
+    <child link="end_effector_link"/>
+    <origin xyz="${link_length} 0 0" rpy="0 ${pi/2} 0"/>
+  </joint>
+  <link name="end_effector_link">
+    <visual>
+      <origin xyz="0 0 0" rpy="0 0 0"/>
+      <geometry>
+	<mesh filename="package://chimera_ros/meshes/end_effector_no_bricks.dae" scale="1 1 1" />
+      </geometry>
+    </visual>
+  </link>
   <joint name="docking_mechanism_dragon_joint" type="fixed">
     <parent link="link1"/>

File: urdf/chimera_bricks_detaching.urdf.xacro (robot description, xacro)
@@ -4,5 +4,5 @@
   <!--<xacro:arg name="fixed_grapple" default="true" />-->
   <!-- spot -->
-  <xacro:include filename="$(find chimera_ros)/urdf/spot.urdf.xacro" />
+  <xacro:include filename="$(find chimera_ros)/urdf/spot_dock.urdf.xacro" />
   <!-- free arm -->
   <xacro:include filename="$(find dragon)/robots/quad/euclid_201709.urdf.xacro" />
@@ -10,19 +10,32 @@
   <joint name="grapple_attachment_joint" type="fixed">
     <!-- <origin xyz="0.0 0.0 0.224" rpy="${pi} ${pi/2} 0" /> -->
-    <origin xyz="0.0 0.0 0.0" rpy="0 ${-pi/2} 0" />
+    <origin xyz="1.38 0.3 1.29" rpy="${0} ${pi/2} 0" />
     <axis xyz="1 0 0" />
     <parent link="base_fixture" />
     <child link="root" />
   </joint>
-  <joint name="end_effector_fixed_joint" type="fixed">
-    <parent link="link4"/>
-    <child link="end_effector_link"/>
-    <origin xyz="${link_length} 0 0" rpy="${0} ${pi/2} ${0}"/>
+  <!-- <joint name="end_effector_fixed_joint" type="fixed"> -->
+  <!--   <parent link="link4"/> -->
+  <!--   <child link="end_effector_link"/> -->
+  <!--   <origin xyz="${link_length} 0 0" rpy="${0} ${pi/2} ${0}"/> -->
+  <!-- </joint> -->
+  <!-- <link name="end_effector_link"> -->
+  <!--   <visual> -->
+  <!--     <origin xyz="0 0 0" rpy="0 0 0"/> -->
+  <!--     <geometry> -->
+  <!-- 	<mesh filename="package://chimera_ros/meshes/end_effector.dae" scale="1 1 1" /> -->
+  <!--     </geometry> -->
+  <!--   </visual> -->
+  <!-- </link> -->
+  <joint name="docking_mechanism_dragon_joint" type="fixed">
+    <parent link="link1"/>
+    <child link="docking_mechanism_dragon_link"/>
+    <origin xyz="${-link_length/2 + 0.15} 0.005 0" rpy="0 ${pi/2} 0"/>
   </joint>
-  <link name="end_effector_link">
+  <link name="docking_mechanism_dragon_link">
     <visual>
       <origin xyz="0 0 0" rpy="0 0 0"/>
       <geometry>
-	<mesh filename="package://chimera_ros/meshes/end_effector.dae" scale="1 1 1" />
+	<mesh filename="package://chimera_ros/meshes/docking_mechanism_dragon_side.dae" scale="0.18 0.18 0.18" />
       </geometry>
     </visual>

File: urdf/chimera_bricks_docking.urdf.xacro (robot description, xacro)
@@ -5,5 +5,5 @@
   <!--<xacro:arg name="fixed_grapple" default="true" />-->
   <!-- spot -->
-  <xacro:include filename="$(find chimera_ros)/urdf/spot.urdf.xacro" />
+  <xacro:include filename="$(find chimera_ros)/urdf/spot_dock.urdf.xacro" />
   <!-- free arm -->
   <xacro:include filename="$(find dragon)/robots/quad/euclid_201709.urdf.xacro" />
@@ -38,7 +38,20 @@
      <origin xyz="0 0 0" rpy="0 0 0"/>
      <geometry>
-       <mesh filename="package://chimera_ros/meshes/end_effector.dae" scale="1 1 1" />
+       <mesh filename="package://chimera_ros/meshes/end_effector_no_bricks.dae" scale="1 1 1" />
      </geometry>
     </visual>
   </link>
+  <joint name="docking_mechanism_dragon_joint" type="fixed">
+    <parent link="link1"/>
+    <child link="docking_mechanism_dragon_link"/>
+    <origin xyz="${-link_length/2 + 0.15} 0.005 0" rpy="0 ${pi/2} 0"/>
+  </joint>
+  <link name="docking_mechanism_dragon_link">
+    <visual>
+      <origin xyz="0 0 0" rpy="0 0 0"/>
+      <geometry>
+	<mesh filename="package://chimera_ros/meshes/docking_mechanism_dragon_side.dae" scale="0.18 0.18 0.18" />
+      </geometry>
+    </visual>
+  </link>
 </robot>
